Commit message: feat: colony_manipulation (Aşama 4) MoveIt entegrasyonu
- worker.urdf.xacro: 3-DOF robotik kol ve gripper eklendi
- URDF içine Ignition ros2_control (JointTrajectoryController) tanımlandı
- colony_manipulation paketi oluşturuldu
- SRDF (worker.srdf), kinematik (KDL), joint limits ve controller yapılandırmaları yapıldı
- move_group.launch.py eklendi
- Aşama 4 (%100) tamamlandı, proje %59'a ulaştı.

File: src/colony_description/urdf/worker.urdf.xacro (robot description, xacro)
@@ -147,3 +147,108 @@
     </sensor>
   </gazebo>
+  <!-- ============================================== -->
+  <!-- 5. 3-DOF ARM & GRIPPER                         -->
+  <!-- ============================================== -->
+  <link name="arm_base_link">
+    <visual>
+      <geometry><box size="0.1 0.1 0.1"/></geometry>
+      <material name="black"/>
+    </visual>
+    <collision><geometry><box size="0.1 0.1 0.1"/></geometry></collision>
+    <inertial><mass value="1.0"/><inertia ixx="0.01" ixy="0" ixz="0" iyy="0.01" iyz="0" izz="0.01"/></inertial>
+  </link>
+  <joint name="arm_base_joint" type="fixed">
+    <parent link="base_link"/>
+    <child link="arm_base_link"/>
+    <origin xyz="0.1 0 0.15" rpy="0 0 0"/>
+  </joint>
+  <link name="shoulder_link">
+    <visual>
+      <geometry><cylinder radius="0.05" length="0.1"/></geometry>
+      <material name="gray"/>
+    </visual>
+    <collision><geometry><cylinder radius="0.05" length="0.1"/></geometry></collision>
+    <inertial><mass value="1.0"/><inertia ixx="0.01" ixy="0" ixz="0" iyy="0.01" iyz="0" izz="0.01"/></inertial>
+  </link>
+  <joint name="joint1" type="revolute">
+    <parent link="arm_base_link"/>
+    <child link="shoulder_link"/>
+    <origin xyz="0 0 0.05" rpy="0 0 0"/>
+    <axis xyz="0 0 1"/>
+    <limit lower="-1.57" upper="1.57" effort="10.0" velocity="1.0"/>
+  </joint>
+  <link name="upper_arm_link">
+    <visual>
+      <geometry><box size="0.05 0.05 0.3"/></geometry>
+      <origin xyz="0 0 0.15" rpy="0 0 0"/>
+      <material name="gray"/>
+    </visual>
+    <collision><geometry><box size="0.05 0.05 0.3"/></geometry><origin xyz="0 0 0.15" rpy="0 0 0"/></collision>
+    <inertial><mass value="1.0"/><origin xyz="0 0 0.15" rpy="0 0 0"/><inertia ixx="0.01" ixy="0" ixz="0" iyy="0.01" iyz="0" izz="0.01"/></inertial>
+  </link>
+  <joint name="joint2" type="revolute">
+    <parent link="shoulder_link"/>
+    <child link="upper_arm_link"/>
+    <origin xyz="0 0 0.05" rpy="0 0 0"/>
+    <axis xyz="0 1 0"/>
+    <limit lower="-1.57" upper="1.57" effort="10.0" velocity="1.0"/>
+  </joint>
+  <link name="forearm_link">
+    <visual>
+      <geometry><box size="0.05 0.05 0.2"/></geometry>
+      <origin xyz="0 0 0.1" rpy="0 0 0"/>
+      <material name="gray"/>
+    </visual>
+    <collision><geometry><box size="0.05 0.05 0.2"/></geometry><origin xyz="0 0 0.1" rpy="0 0 0"/></collision>
+    <inertial><mass value="0.5"/><origin xyz="0 0 0.1" rpy="0 0 0"/><inertia ixx="0.01" ixy="0" ixz="0" iyy="0.01" iyz="0" izz="0.01"/></inertial>
+  </link>
+  <joint name="joint3" type="revolute">
+    <parent link="upper_arm_link"/>
+    <child link="forearm_link"/>
+    <origin xyz="0 0 0.3" rpy="0 0 0"/>
+    <axis xyz="0 1 0"/>
+    <limit lower="-1.57" upper="1.57" effort="10.0" velocity="1.0"/>
+  </joint>
+  <!-- Dummy Gripper Link (End Effector) -->
+  <link name="gripper_link">
+    <visual>
+      <geometry><box size="0.1 0.1 0.05"/></geometry>
+      <material name="blue"/>
+    </visual>
+    <collision><geometry><box size="0.1 0.1 0.05"/></geometry></collision>
+    <inertial><mass value="0.1"/><inertia ixx="0.001" ixy="0" ixz="0" iyy="0.001" iyz="0" izz="0.001"/></inertial>
+  </link>
+  <joint name="gripper_fixed_joint" type="fixed">
+    <parent link="forearm_link"/>
+    <child link="gripper_link"/>
+    <origin xyz="0 0 0.225" rpy="0 0 0"/>
+  </joint>
+  <!-- ============================================== -->
+  <!-- 6. ROS2 CONTROL (IGNITION)                     -->
+  <!-- ============================================== -->
+  <ros2_control name="IgnitionSystem" type="system">
+    <hardware>
+      <plugin>ign_ros2_control/IgnitionSystem</plugin>
+    </hardware>
+    <joint name="joint1">
+      <command_interface name="position"/>
+      <state_interface name="position"/>
+      <state_interface name="velocity"/>
+    </joint>
+    <joint name="joint2">
+      <command_interface name="position"/>
+      <state_interface name="position"/>
+      <state_interface name="velocity"/>
+    </joint>
+    <joint name="joint3">
+      <command_interface name="position"/>
+      <state_interface name="position"/>
+      <state_interface name="velocity"/>
+    </joint>
+  </ros2_control>
+  <gazebo>
+    <plugin filename="ign_ros2_control-system" name="ign_ros2_control::IgnitionROS2ControlPlugin">
+      <parameters>$(find colony_manipulation)/config/controllers.yaml</parameters>
+    </plugin>
+  </gazebo>
 </robot>
